Commit message: 1,update movegroup

File: polishingrobot_description/urdf/polishingrobot_description.urdf (robot description, URDF)
Before this commit: robot polishingrobot_description, 15 links, 14 joints
Links:
- added link world
Joints:
- added joint map_joint: type fixed, parent world, child map, origin xyz=0.0 0.0 0.0 rpy=0.0 0.0 0.0

Commit message: 1,update cplus aubo control

File: polishingrobot_description/urdf/polishingrobot_description.urdf (robot description, URDF)
Before this commit: robot polishingrobot_description, 16 links, 15 joints
Joints:
- joint wrist3_joint: limit lower=-3.05 upper=3.05 effort=0 velocity=0 -> lower=-3.05 upper=0.55 effort=0 velocity=0
